Commit message: New errors

File: dual_arm_robot_setup/src/fr3_dual_arm_sim/urdf/dual_fr3.xacro (robot description, xacro)
@@ -1,43 +1,34 @@
 <?xml version="1.0"?>
-<robot xmlns:xacro="http://ros.org/wiki/xacro" name="dual_fr3">
-  <xacro:include filename="$(find franka_description)/robots/fr3/fr3.urdf.xacro"/>
-  <group ns="fr3_a">
-    <xacro:fr3
-      prefix="fr3_a/"
-      add_base_link="true"
-      use_gazebo_control="true"
-      />
-  </group>
-  <!-- Second arm -->
-  <group ns="fr3_b">
-    <xacro:fr3
-      prefix="fr3_b/"
-      add_base_link="true"
-      use_gazebo_control="true"
-      />
-  </group>
-  <link name="fr3_a_base">
-  </link>
-  <joint name="fr3_a_base_joint" type="fixed">
-    <parent link="world"/>
-    <child link="fr3_a_base"/>
-    <origin xyz="0.5 0.3 0.75" rpy="0 0 0"/>
-  </joint>
-  <joint name="fr3_a_to_robot" type="fixed">
-    <parent link="fr3_a_base"/>
-    <child link="fr3_a_base_link"/>
-    <origin xyz="0 0 0" rpy="0 0 0"/>
-  </joint>
-  <link name="fr3_b_base">
-  </link>
-  <joint name="fr3_b_base_joint" type="fixed">
-    <parent link="world"/>
-    <child link="fr3_b_base"/>
-    <origin xyz="-0.5 -0.3 0.75" rpy="0 0 0"/>
-  </joint>
-  <joint name="fr3_b_to_robot" type="fixed">
-    <parent link="fr3_b_base"/>
-    <child link="fr3_b_base_link"/>
-    <origin xyz="0 0 0" rpy="0 0 0"/>
-  </joint>
+<robot xmlns:xacro="http://www.ros.org/wiki/xacro" name="dual_fr3">
+  <!-- Include FR3 wrapper -->
+  <xacro:include filename="$(find franka_description)/robots/fr3/fr3.urdf.xacro" />
+  <!-- Macro to spawn one FR3 with prefix -->
+  <xacro:macro name="spawn_fr3" params="prefix parent_link *origin">
+    <joint name="${prefix}_world_joint" type="fixed">
+      <xacro:insert_block name="origin"/>
+      <parent link="${parent_link}"/>
+      <child link="${prefix}fr3_link0"/>
+    </joint>
+    <!-- Call the franka_robot wrapper -->
+    <xacro:franka_robot
+        arm_id="fr3"
+        arm_prefix="${prefix}"
+        description_pkg="franka_description"
+        joint_limits="${xacro.load_yaml('$(find franka_description)/robots/fr3/joint_limits.yaml')}"
+        inertials="${xacro.load_yaml('$(find franka_description)/robots/fr3/inertials.yaml')}"
+        kinematics="${xacro.load_yaml('$(find franka_description)/robots/fr3/kinematics.yaml')}"
+        dynamics="${xacro.load_yaml('$(find franka_description)/robots/fr3/dynamics.yaml')}"
+        safety_distance="0.03"
+        with_sc="false"
+        gazebo="false"
+        connected_to=""/>
+  </xacro:macro>
+  <!-- Left arm -->
+  <xacro:spawn_fr3 prefix="left" parent_link="base">
+    <origin xyz="0 0.4 0" rpy="0 0 0"/>
+  </xacro:spawn_fr3>
+  <!-- Right arm -->
+  <xacro:spawn_fr3 prefix="right" parent_link="base">
+    <origin xyz="0 -0.4 0" rpy="0 0 0"/>
+  </xacro:spawn_fr3>
 </robot>

Commit message: Spawn two arms and table in gazebo

File: dual_arm_robot_setup/src/fr3_dual_arm_sim/urdf/dual_fr3.xacro (robot description, xacro)
@@ -1,14 +1,38 @@
 <?xml version="1.0"?>
 <robot xmlns:xacro="http://www.ros.org/wiki/xacro" name="dual_fr3">
-  <!-- Include FR3 wrapper -->
-  <xacro:include filename="$(find franka_description)/robots/fr3/fr3.urdf.xacro" />
-  <!-- Macro to spawn one FR3 with prefix -->
+  <link name="world"/>
+  <joint name="world_to_base_joint" type="fixed">
+    <parent link="world"/>
+    <child link="base_link"/>
+    <origin xyz="0 0 0" rpy="0 0 0"/>
+  </joint>
+  <link name="base_link">
+    <inertial>
+      <mass value="50.0"/>
+      <origin xyz="0 0 0" rpy="0 0 0"/>
+      <inertia ixx="1.0" ixy="0" ixz="0" iyy="1.0" iyz="0" izz="1.0"/>
+    </inertial>
+    <visual name="visual">
+      <origin rpy="1.5708 0.0 -1.5708" xyz="1.25 0.75 0.0"/>
+      <geometry>
+        <mesh filename="package://fr3_dual_arm_sim/models/table_with_pedestal/meshes/table_with_pedestal.STL" scale="0.001 0.001 0.001"/>
+      </geometry>
+      <material name="Grey">
+        <color rgba="0.7 0.7 0.7 1"/>
+      </material>
+    </visual>
+    <collision name="collision">
+      <geometry>
+        <mesh filename="package://fr3_dual_arm_sim/models/table_with_pedestal/meshes/table_with_pedestal.STL" scale="0.001 0.001 0.001"/>
+      </geometry>
+    </collision>
+  </link>
+  <xacro:include filename="$(find franka_description)/robots/common/franka_robot.xacro" />
   <xacro:macro name="spawn_fr3" params="prefix parent_link *origin">
-    <joint name="${prefix}_world_joint" type="fixed">
+    <joint name="${prefix}base_to_arm_joint" type="fixed">
       <xacro:insert_block name="origin"/>
       <parent link="${parent_link}"/>
       <child link="${prefix}fr3_link0"/>
     </joint>
-    <!-- Call the franka_robot wrapper -->
     <xacro:franka_robot
         arm_id="fr3"
@@ -24,11 +48,9 @@
         connected_to=""/>
   </xacro:macro>
-  <!-- Left arm -->
-  <xacro:spawn_fr3 prefix="left" parent_link="base">
-    <origin xyz="0 0.4 0" rpy="0 0 0"/>
+  <xacro:spawn_fr3 prefix="left_" parent_link="base_link">
+    <origin xyz="-0.07 0.4 0.84" rpy="0 0 3.14159"/>
   </xacro:spawn_fr3>
-  <!-- Right arm -->
-  <xacro:spawn_fr3 prefix="right" parent_link="base">
-    <origin xyz="0 -0.4 0" rpy="0 0 0"/>
+  <xacro:spawn_fr3 prefix="right_" parent_link="base_link">
+    <origin xyz="-0.07 -0.5 0.84" rpy="0 0 3.14159"/>
   </xacro:spawn_fr3>
 </robot>
