Commit message: Add grippers, remove table STL and modify moveit

File: dual_arm_robot_setup/src/fr3_dual_arm_moveit_config/config/dual_fr3.ros2_control.xacro (robot description, xacro)
@@ -106,4 +106,18 @@
                 <state_interface name="velocity"/>
             </joint>
+            <joint name="left_fr3_finger_joint1">
+                <command_interface name="position"/>
+                <state_interface name="position">
+                  <param name="initial_value">${initial_positions['left_fr3_finger_joint1']}</param>
+                </state_interface>
+                <state_interface name="velocity"/>
+            </joint>
+            <joint name="right_fr3_finger_joint1">
+                <command_interface name="position"/>
+                <state_interface name="position">
+                  <param name="initial_value">${initial_positions['right_fr3_finger_joint1']}</param>
+                </state_interface>
+                <state_interface name="velocity"/>
+            </joint>
         </ros2_control>
     </xacro:macro>

File: dual_arm_robot_setup/src/fr3_dual_arm_sim/urdf/dual_fr3.urdf (robot description, URDF)
Before this commit: robot dual_fr3, 20 links, 19 joints
Links:
- removed link base_link
- added link base; collision box size=0.9 1.6 1.68; visual box size=0.9 1.6 1.68
- added link left_fr3_hand, mass 0.6544; collision mesh filename=package://franka_description/meshes/robot_ee/franka_hand_wh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; visual mesh filename=package://franka_description/meshes/robot_ee/franka_hand_wh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
- added link left_fr3_hand_sc
- added link left_fr3_hand_tcp
- added link left_fr3_leftfinger, mass 0.0291; collision box size=17.5e-3 15.2e-3 18.5e-3; collision box size=17.5e-3 7e-3 23.5e-3
- added link left_fr3_link0_sc
- added link left_fr3_link1_sc
- added link left_fr3_link2_sc
- added link left_fr3_link3_sc
- added link left_fr3_link4_sc
- added link left_fr3_link5_sc
- added link left_fr3_link6_sc
- added link left_fr3_link7_sc
- added link left_fr3_rightfinger, mass 0.0291; collision box size=17.5e-3 15.2e-3 18.5e-3; collision box size=17.5e-3 7e-3 23.5e-3
- added link right_fr3_hand, mass 0.6544; collision mesh filename=package://franka_description/meshes/robot_ee/franka_hand_wh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; visual mesh filename=package://franka_description/meshes/robot_ee/franka_hand_wh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
- added link right_fr3_hand_sc
- added link right_fr3_hand_tcp
- added link right_fr3_leftfinger, mass 0.0291; collision box size=17.5e-3 15.2e-3 18.5e-3; collision box size=17.5e-3 7e-3 23.5e-3
- added link right_fr3_link0_sc
- added link right_fr3_link1_sc
- added link right_fr3_link2_sc
- added link right_fr3_link3_sc
- added link right_fr3_link4_sc
- added link right_fr3_link5_sc
- added link right_fr3_link6_sc
- added link right_fr3_link7_sc
- added link right_fr3_rightfinger, mass 0.0291; collision box size=17.5e-3 15.2e-3 18.5e-3; collision box size=17.5e-3 7e-3 23.5e-3
Joints:
- removed joint world_to_base_joint
- added joint fixed: type fixed, parent world, child base
- added joint left_fr3_finger_joint1: type prismatic, parent left_fr3_hand, child left_fr3_leftfinger, origin xyz=0 0 0.0584 rpy=0 0 0, axis 0 1 0, limit lower=0.0 upper=0.04 effort=100 velocity=0.2
- added joint left_fr3_finger_joint2: type prismatic, parent left_fr3_hand, child left_fr3_rightfinger, origin xyz=0 0 0.0584 rpy=0 0 3.141592653589793, axis 0 1 0, limit lower=0.0 upper=0.04 effort=100 velocity=0.2, mimic joint=left_fr3_finger_joint1
- added joint left_fr3_hand_joint: type fixed, parent left_fr3_link8, child left_fr3_hand, origin xyz=0 0 0 rpy=0 0 -0.7853981633974483
- added joint left_fr3_hand_sc_joint: type fixed, parent left_fr3_hand, child left_fr3_hand_sc, origin rpy=0 0 0
- added joint left_fr3_hand_tcp_joint: type fixed, parent left_fr3_hand, child left_fr3_hand_tcp, origin xyz=0 0 0.1034 rpy=0 0 0
- added joint left_fr3_link0_sc_joint: type fixed, parent left_fr3_link0, child left_fr3_link0_sc, origin rpy=0 0 0
- added joint left_fr3_link1_sc_joint: type fixed, parent left_fr3_link1, child left_fr3_link1_sc, origin rpy=0 0 0
- added joint left_fr3_link2_sc_joint: type fixed, parent left_fr3_link2, child left_fr3_link2_sc, origin rpy=0 0 0
- added joint left_fr3_link3_sc_joint: type fixed, parent left_fr3_link3, child left_fr3_link3_sc, origin rpy=0 0 0
- added joint left_fr3_link4_sc_joint: type fixed, parent left_fr3_link4, child left_fr3_link4_sc, origin rpy=0 0 0
- added joint left_fr3_link5_sc_joint: type fixed, parent left_fr3_link5, child left_fr3_link5_sc, origin rpy=0 0 0
- added joint left_fr3_link6_sc_joint: type fixed, parent left_fr3_link6, child left_fr3_link6_sc, origin rpy=0 0 0
- added joint left_fr3_link7_sc_joint: type fixed, parent left_fr3_link7, child left_fr3_link7_sc, origin rpy=0 0 0.7853981633974483
- added joint right_fr3_finger_joint1: type prismatic, parent right_fr3_hand, child right_fr3_leftfinger, origin xyz=0 0 0.0584 rpy=0 0 0, axis 0 1 0, limit lower=0.0 upper=0.04 effort=100 velocity=0.2
- added joint right_fr3_finger_joint2: type prismatic, parent right_fr3_hand, child right_fr3_rightfinger, origin xyz=0 0 0.0584 rpy=0 0 3.141592653589793, axis 0 1 0, limit lower=0.0 upper=0.04 effort=100 velocity=0.2, mimic joint=right_fr3_finger_joint1
- added joint right_fr3_hand_joint: type fixed, parent right_fr3_link8, child right_fr3_hand, origin xyz=0 0 0 rpy=0 0 -0.7853981633974483
- added joint right_fr3_hand_sc_joint: type fixed, parent right_fr3_hand, child right_fr3_hand_sc, origin rpy=0 0 0
- added joint right_fr3_hand_tcp_joint: type fixed, parent right_fr3_hand, child right_fr3_hand_tcp, origin xyz=0 0 0.1034 rpy=0 0 0
- added joint right_fr3_link0_sc_joint: type fixed, parent right_fr3_link0, child right_fr3_link0_sc, origin rpy=0 0 0
- added joint right_fr3_link1_sc_joint: type fixed, parent right_fr3_link1, child right_fr3_link1_sc, origin rpy=0 0 0
- added joint right_fr3_link2_sc_joint: type fixed, parent right_fr3_link2, child right_fr3_link2_sc, origin rpy=0 0 0
- added joint right_fr3_link3_sc_joint: type fixed, parent right_fr3_link3, child right_fr3_link3_sc, origin rpy=0 0 0
- added joint right_fr3_link4_sc_joint: type fixed, parent right_fr3_link4, child right_fr3_link4_sc, origin rpy=0 0 0
- added joint right_fr3_link5_sc_joint: type fixed, parent right_fr3_link5, child right_fr3_link5_sc, origin rpy=0 0 0
- added joint right_fr3_link6_sc_joint: type fixed, parent right_fr3_link6, child right_fr3_link6_sc, origin rpy=0 0 0
- added joint right_fr3_link7_sc_joint: type fixed, parent right_fr3_link7, child right_fr3_link7_sc, origin rpy=0 0 0.7853981633974483
- joint left_base_to_arm_joint: parent base_link -> base
- joint right_base_to_arm_joint: parent base_link -> base
